File: TimeMachine.sch (KiCad schematic (older format))
At the start: 51 parts, among them J1 AppleIIBus, J2 JTAG, U1 EPM7128SL84, U2 DS1215, U3 74AHCT04, U4 AS6C8008, U5 39F040, Y1 32k768

Commit message: Trying this on reworked boards
Parts:
- R3: value 100 -> 15
Changed lines of the file:
@@
 P 1350 1600
 F 0 "R3" V 1200 1600 50  0000 C CNN
-F 1 "100" V 1300 1600 50  0000 C BNN
+F 1 "15" V 1300 1600 50  0000 C BNN
 F 2 "stdpads:R_0805" H 1350 1600 50  0001 C CNN
 F 3 "~" H 1350 1600 50  0001 C CNN
@@
 Text Label 2800 1500 2    50   ~ 0
 ~INH~
-Wire Bus Line
-	2300 600  2300 2800
-Wire Bus Line
-	2400 4200 2400 5700
-Wire Bus Line
-	4800 600  4800 3300
-Wire Bus Line
-	6600 3600 6600 5600
-Wire Bus Line
-	6700 3300 6700 4800
-Wire Bus Line
-	8300 3500 8300 6100
-Wire Bus Line
-	6200 3500 6200 6100
-Wire Bus Line
-	2300 3300 2300 6100
-Wire Bus Line
-	600  700  600  4300
-Wire Bus Line
-	4600 700  4600 2800
-Wire Bus Line
-	2000 2800 2000 4300
-Wire Bus Line
-	4700 3600 4700 5700
 $Comp
 L power:GND #PWR?
@@
 	1    0    0    -1
 $EndComp
+Wire Bus Line
+	2300 600  2300 2800
+Wire Bus Line
+	2400 4200 2400 5700
+Wire Bus Line
+	4800 600  4800 3300
+Wire Bus Line
+	6600 3600 6600 5600
+Wire Bus Line
+	6700 3300 6700 4800
+Wire Bus Line
+	8300 3500 8300 6100
+Wire Bus Line
+	6200 3500 6200 6100
+Wire Bus Line
+	2300 3300 2300 6100
+Wire Bus Line
+	600  700  600  4300
+Wire Bus Line
+	4600 700  4600 2800
+Wire Bus Line
+	2000 2800 2000 4300
+Wire Bus Line
+	4700 3600 4700 5700
 $EndSCHEMATC

Commit message: Fixed mistake, submitted to JLCPCB
Parts:
- Y1: footprint Crystal_C26-LF_D2.1mm_L6.5mm_Horizontal_1EP_style1 -> Crystal:Crystal_C26-LF_D2.1mm_L6.5mm_Horizontal; symbol Device:Crystal_GND3_Small -> Device:Crystal_Small
Connections:
- net GND: no longer U3.13, Y1.3
- net R~W~: now also U3.13; no longer U3.3
- net ~OE~: now also U3.12; no longer U2.12 (~OE~), U3.4
- net CA2 renamed DS~WE~
- net DS~WE~: now also U3.3
- new net DS~OE~: U2.12 (~OE~), U3.4
- no-connect marks 7 -> 6
Other:
- moved on the sheet: U3A, U3F

Commit message: Switched schematic to new GW libraries
Parts:
- U1: symbol stdparts:EPM7128SL84 -> GW_PLD:EPM7128SL84
- U2: symbol stdparts:DS1215 -> GW_Digital:DS1215
- U4: symbol stdparts:AS6C8008 -> GW_RAM:SRAM-1Mx8-TSOP2-44
- U5: symbol stdparts:39F040 -> GW_RAM:Flash-512Kx8-PLCC-32
Changed lines of the file:
@@
 	1    0    0    -1
 $EndComp
-Text Label 5900 5500 0    50   ~ 0
+Text Label 5900 5400 0    50   ~ 0
 RAMCS
-Text Label 6400 5400 1    50   ~ 0
+Text Label 6400 5300 1    50   ~ 0
 RAMROM~CS~g
 $Comp
-L stdparts:AS6C8008 U4
+L GW_RAM:SRAM-1Mx8-TSOP2-44 U4
 U 1 1 5D7A1D1B
 P 5500 4850
@@
 $EndComp
 $Comp
-L stdparts:39F040 U5
+L GW_RAM:Flash-512Kx8-PLCC-32 U5
 U 1 1 5D81337E
-P 7500 4800
-F 0 "U5" H 7500 5850 50  0000 C CNN
-F 1 "39F040" V 7500 4800 50  0000 C CNN
-F 2 "stdpads:PLCC-32_SMDSocket" H 7500 4800 50  0001 C CNN
-F 3 "http://ww1.microchip.com/downloads/en/DeviceDoc/25022B.pdf" H 7500 4800 50  0001 C CNN
-	1    7500 4800
+P 7400 4800
+F 0 "U5" H 7400 5850 50  0000 C CNN
+F 1 "39F040" V 7400 4800 50  0000 C CNN
+F 2 "stdpads:PLCC-32_SMDSocket" H 7400 4800 50  0001 C CNN
+F 3 "http://ww1.microchip.com/downloads/en/DeviceDoc/25022B.pdf" H 7400 4800 50  0001 C CNN
+	1    7400 4800
 	1    0    0    -1
 $EndComp
@@
 L power:GND #PWR0107
 U 1 1 5D847F2B
-P 8000 5700
-F 0 "#PWR0107" H 8000 5450 50  0001 C CNN
-F 1 "GND" H 8000 5550 50  0000 C CNN
-F 2 "" H 8000 5700 50  0001 C CNN
-F 3 "" H 8000 5700 50  0001 C CNN
-	1    8000 5700
+P 7800 5700
+F 0 "#PWR0107" H 7800 5450 50  0001 C CNN
+F 1 "GND" H 7800 5550 50  0000 C CNN
+F 2 "" H 7800 5700 50  0001 C CNN
+F 3 "" H 7800 5700 50  0001 C CNN
+	1    7800 5700
 	1    0    0    -1
 $EndComp
@@
 L power:+5V #PWR0113
 U 1 1 5D848386
-P 8000 3900
-F 0 "#PWR0113" H 8000 3750 50  0001 C CNN
-F 1 "+5V" H 8000 4050 50  0000 C CNN
-F 2 "" H 8000 3900 50  0001 C CNN
-F 3 "" H 8000 3900 50  0001 C CNN
-	1    8000 3900
-	1    0    0    -1
-$EndComp
-Text Label 5900 5600 0    50   ~ 0
+P 7800 3900
+F 0 "#PWR0113" H 7800 3750 50  0001 C CNN
+F 1 "+5V" H 7800 4050 50  0000 C CNN
+F 2 "" H 7800 3900 50  0001 C CNN
+F 3 "" H 7800 3900 50  0001 C CNN
+	1    7800 3900
+	1    0    0    -1
+$EndComp
+Text Label 5900 5500 0    50   ~ 0
 R~W~
 Text Label 7000 4300 2    50   ~ 0
@@
 Text Label 1600 4500 0    50   ~ 0
 ~IOSEL~
-Text Label 8000 5400 0    50   ~ 0
+Text Label 7800 5400 0    50   ~ 0
 ~OE~
 $Comp
@@
 Text Label 5900 4500 0    50   ~ 0
 RD7
-Wire Wire Line
-	5900 5700 5900 5800
-Connection ~ 5900 5800
 Text Label 7000 5700 2    50   ~ 0
 RA18
@@
 Text Label 2800 4000 2    50   ~ 0
 RAMCS
-Text Label 8000 4200 0    50   ~ 0
+Text Label 7800 4200 0    50   ~ 0
 RD1
-Text Label 8000 4300 0    50   ~ 0
+Text Label 7800 4300 0    50   ~ 0
 RD2
-Text Label 8000 4400 0    50   ~ 0
+Text Label 7800 4400 0    50   ~ 0
 RD3
-Text Label 8000 4100 0    50   ~ 0
+Text Label 7800 4100 0    50   ~ 0
 RD0
-Text Label 8000 4500 0    50   ~ 0
+Text Label 7800 4500 0    50   ~ 0
 RD4
-Text Label 8000 4600 0    50   ~ 0
+Text Label 7800 4600 0    50   ~ 0
 RD5
-Text Label 8000 4700 0    50   ~ 0
+Text Label 7800 4700 0    50   ~ 0
 RD6
-Text Label 8000 4800 0    50   ~ 0
+Text Label 7800 4800 0    50   ~ 0
 RD7
 $Comp
@@
 	2400 3700 2800 3700
 $Comp
-L stdparts:EPM7128SL84 U1
+L GW_PLD:EPM7128SL84 U1
 U 1 1 5CBA3E53
 P 3550 3000
@@
 	5900 4800 6100 4800
 Entry Wire Line
-	8300 4300 8200 4400
-Entry Wire Line
-	8300 4400 8200 4500
-Entry Wire Line
-	8300 4500 8200 4600
-Entry Wire Line
-	8300 4600 8200 4700
-Entry Wire Line
-	8300 4700 8200 4800
-Entry Wire Line
-	8300 4200 8200 4300
-Entry Wire Line
-	8300 4100 8200 4200
-Entry Wire Line
-	8300 4000 8200 4100
-Wire Wire Line
-	8000 4100 8200 4100
-Wire Wire Line
-	8000 4200 8200 4200
-Wire Wire Line
-	8000 4300 8200 4300
-Wire Wire Line
-	8000 4400 8200 4400
-Wire Wire Line
-	8000 4500 8200 4500
-Wire Wire Line
-	8000 4600 8200 4600
-Wire Wire Line
-	8000 4700 8200 4700
-Wire Wire Line
-	8000 4800 8200 4800
+	8100 4300 8000 4400
+Entry Wire Line
+	8100 4400 8000 4500
+Entry Wire Line
+	8100 4500 8000 4600
+Entry Wire Line
+	8100 4600 8000 4700
+Entry Wire Line
+	8100 4700 8000 4800
+Entry Wire Line
+	8100 4200 8000 4300
+Entry Wire Line
+	8100 4100 8000 4200
+Entry Wire Line
+	8100 4000 8000 4100
+Wire Wire Line
+	7800 4100 8000 4100
+Wire Wire Line
+	7800 4200 8000 4200
+Wire Wire Line
+	7800 4300 8000 4300
+Wire Wire Line
+	7800 4400 8000 4400
+Wire Wire Line
+	7800 4500 8000 4500
+Wire Wire Line
+	7800 4600 8000 4600
+Wire Wire Line
+	7800 4700 8000 4700
+Wire Wire Line
+	7800 4800 8000 4800
 Entry Wire Line
 	4800 3300 4700 3400
@@
 Wire Bus Line
 	2300 6100 6200 6100
-Wire Wire Line
-	6400 5400 6400 2850
 Text Label 7200 2850 2    50   ~ 0
 RAMROM~CS~g
@@
 $EndComp
 $Comp
-L stdparts:DS1215 U2
+L GW_Digital:DS1215 U2
 U 1 1 5D8605F3
 P 6700 2100
@@
 	7300 2850 6400 2850
 Wire Bus Line
-	6200 3500 8300 3500
-Wire Bus Line
 	4700 3600 6600 3600
 Wire Bus Line
-	6200 6100 8300 6100
+	6100 6100 6200 6100
 Connection ~ 6200 6100
 Wire Wire Line
-	5900 5400 6400 5400
-Text Label 8000 5200 0    50   ~ 0
+	5900 5300 6400 5300
+Text Label 7800 5200 0    50   ~ 0
 ROM~CS~
 Wire Bus Line
@@
 Text Label 7200 2150 0    50   ~ 0
 DS~OE~
-Text Label 8000 5300 0    50   ~ 0
+Text Label 7800 5300 0    50   ~ 0
 R~W~
 Text Label 2800 3100 2    50   ~ 0
@@
 Wire Wire Line
 	7900 2450 8500 2450
-Wire Bus Line
-	6600 3600 6600 5600
-Wire Bus Line
-	6700 3300 6700 4800
-Wire Bus Line
-	8300 3500 8300 6100
-Wire Bus Line
-	6200 3500 6200 6100
-Wire Bus Line
-	4700 3600 4700 5700
-Wire Bus Line
-	2400 4200 2400 5700
-Wire Bus Line
-	2300 3300 2300 6100
-Wire Bus Line
-	600  700  600  4300
-Wire Bus Line
-	4600 700  4600 2800
-Wire Bus Line
-	4800 600  4800 3300
-Wire Bus Line
-	2300 600  2300 2800
-Wire Bus Line
-	2000 2800 2000 4300
 $Comp
 L Device:Crystal_Small Y1
@@
 	0    1    1    0
 $EndComp
+Wire Bus Line
+	6200 3500 8100 3500
+Wire Bus Line
+	6200 6100 8100 6100
+Wire Wire Line
+	6400 5300 6400 2850
+Wire Wire Line
+	5900 5600 5900 5800
+Wire Bus Line
+	2300 600  2300 2800
+Wire Bus Line
+	2400 4200 2400 5700
+Wire Bus Line
+	4800 600  4800 3300
+Wire Bus Line
+	6600 3600 6600 5600
+Wire Bus Line
+	6700 3300 6700 4800
+Wire Bus Line
+	8100 3500 8100 6100
+Wire Bus Line
+	6200 3500 6200 6100
+Wire Bus Line
+	2300 3300 2300 6100
+Wire Bus Line
+	600  700  600  4300
+Wire Bus Line
+	4600 700  4600 2800
+Wire Bus Line
+	2000 2800 2000 4300
+Wire Bus Line
+	4700 3600 4700 5700
+Connection ~ 5900 5800
 $EndSCHEMATC

Commit message: Changed libraries
Parts:
- C1, C12, C14, C15, C16, C18, C19, C2, C20, C21, C24, C25, C26, C3, C4, C5, C6, C7, C8, C9: value 100n -> 2u2
- C10, C11, C17: value 33u -> DNP
- U2: value DS1215 -> DS1315S-5; symbol GW_Digital:DS1215 -> GW_Digital:DS1315
Connections:
- wire segments 212 -> 216
Other:
- moved on the sheet: BT1, FID1, FID2, FID3, FID4, FID5, H1, H2, H3, H4, H5, JP2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
