File: TimeMachine.kicad_pcb (KiCad board)
At the start: 4 copper layers, 107.6 x 59.8 mm, 51 parts, among them J1 AppleIIBus, J2 JTAG, U1 EPM7128SL84, U2 DS1215, U3 74AHCT04, U4 AS6C8008, U5 39F040, Y1 32k768

Commit message: Changed libraries
Parts:
- C1, C12, C14, C15, C16, C18, C19, C2, C20, C21, C24, C25, C26, C3, C4, C5, C6, C7, C8, C9: value 100n -> 2u2
- C10, C11, C17: value 33u -> DNP
Changed lines of the file:
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@@
     (pad 14 smd roundrect (at 2.475 -3.81) (size 1.95 0.6) (layers F.Cu F.Paste F.Mask) (roundrect_rratio 0.25)
       (net 1 +5V))
-    (model ${KISYS3DMOD}/Package_SO.3dshapes/SOIC-14_3.9x8.7mm_P1.27mm.wrl
+    (model ${KISYS3DMOD}/Package_SO.3dshapes/SOIC-14_3.9x8.7mm_P1.27mm.step
       (at (xyz 0 0 0))
       (scale (xyz 1 1 1))
@@
       (effects (font (size 0.8128 0.8128) (thickness 0.1524)))
     )
-    (fp_text value 100n (at 0 0.9) (layer F.Fab) hide
+    (fp_text value 2u2 (at 0 0.9) (layer F.Fab) hide
       (effects (font (size 0.127 0.127) (thickness 0.03175)))
     )
@@
       (effects (font (size 0.8128 0.8128) (thickness 0.1524)))
     )
-    (fp_text value 100n (at 0 0.9) (layer F.Fab) hide
+    (fp_text value 2u2 (at 0 0.9) (layer F.Fab) hide
       (effects (font (size 0.127 0.127) (thickness 0.03175)))
     )
@@
       (effects (font (size 0.8128 0.8128) (thickness 0.1524)))
     )
-    (fp_text value 100n (at 0 0.9) (layer F.Fab) hide
+    (fp_text value 2u2 (at 0 0.9) (layer F.Fab) hide
       (effects (font (size 0.127 0.127) (thickness 0.03175)))
     )
@@
       (effects (font (size 0.8128 0.8128) (thickness 0.1524)))
     )
-    (fp_text value 100n (at 0 0.9) (layer F.Fab) hide
+    (fp_text value 2u2 (at 0 0.9) (layer F.Fab) hide
       (effects (font (size 0.127 0.127) (thickness 0.03175)))
     )
@@
     (pad 2 smd roundrect (at 1.655 1.27) (size 2.51 1) (layers F.Cu F.Paste F.Mask) (roundrect_rratio 0.25)
       (net 71 /RA11))
-    (model ${KISYS3DMOD}/Connector_PinHeader_2.54mm.3dshapes/PinHeader_1x02_P2.54mm_Vertical_SMD_Pin1Left.wrl
-      (at (xyz 0 0 0))
-      (scale (xyz 1 1 1))
-      (rotate (xyz 0 0 0))
-    )
   )
   (module stdpads:IDC_SMD_2x05_P2.54mm_Vertical (layer F.Cu)
@@
     (pad 2 smd roundrect (at 2.52 -5.08) (size 3 1) (layers F.Cu F.Paste F.Mask) (roundrect_rratio 0.25)
       (net 2 GND))
-    (model ${KISYS3DMOD}/Connector_IDC.3dshapes/IDC-Header_2x05_P2.54mm_Vertical.wrl
-      (offset (xyz -1.27 5.08 0))
-      (scale (xyz 1 1 1))
-      (rotate (xyz 0 0 0))
-    )
   )
   (module stdpads:Fiducial (layer F.Cu)
@@
       (effects (font (size 0.8128 0.8128) (thickness 0.1524)))
     )
-    (fp_text value 100n (at 0 0.9) (layer F.Fab) hide
+    (fp_text value 2u2 (at 0 0.9) (layer F.Fab) hide
       (effects (font (size 0.127 0.127) (thickness 0.03175)))
     )
@@
       (effects (font (size 0.8128 0.8128) (thickness 0.1524)))
     )
-    (fp_text value 100n (at 0 0.9) (layer F.Fab) hide
+    (fp_text value 2u2 (at 0 0.9) (layer F.Fab) hide
       (effects (font (size 0.127 0.127) (thickness 0.03175)))
     )
@@
       (effects (font (size 0.8128 0.8128) (thickness 0.1524)))
     )
-    (fp_text value 100n (at 0 0.9) (layer F.Fab) hide
+    (fp_text value 2u2 (at 0 0.9) (layer F.Fab) hide
       (effects (font (size 0.127 0.127) (thickness 0.03175)))
     )
@@
       (effects (font (size 0.8128 0.8128) (thickness 0.1524)))
     )
-    (fp_text value 100n (at 0 0.9) (layer F.Fab) hide
+    (fp_text value 2u2 (at 0 0.9) (layer F.Fab) hide
       (effects (font (size 0.127 0.127) (thickness 0.03175)))
     )
@@
       (effects (font (size 0.8128 0.8128) (thickness 0.1524)))
     )
-    (fp_text value 100n (at 0 0.9) (layer F.Fab) hide
+    (fp_text value 2u2 (at 0 0.9) (layer F.Fab) hide
       (effects (font (size 0.127 0.127) (thickness 0.03175)))
     )
@@
       (effects (font (size 0.8128 0.8128) (thickness 0.1524)))
     )
-    (fp_text value 100n (at 0 0.9) (layer F.Fab) hide
+    (fp_text value 2u2 (at 0 0.9) (layer F.Fab) hide
       (effects (font (size 0.127 0.127) (thickness 0.03175)))
     )
@@
       (effects (font (size 0.8128 0.8128) (thickness 0.1524)))
     )
-    (fp_text value 100n (at 0 0.9) (layer F.Fab) hide
+    (fp_text value 2u2 (at 0 0.9) (layer F.Fab) hide
       (effects (font (size 0.127 0.127) (thickness 0.03175)))
     )
@@
       (effects (font (size 0.8128 0.8128) (thickness 0.1524)))
     )
-    (fp_text value 100n (at 0 0.9) (layer F.Fab) hide
+    (fp_text value 2u2 (at 0 0.9) (layer F.Fab) hide
       (effects (font (size 0.127 0.127) (thickness 0.03175)))
     )
@@
       (effects (font (size 0.8128 0.8128) (thickness 0.1524)))
     )
-    (fp_text value 100n (at 0 0.9) (layer F.Fab) hide
+    (fp_text value 2u2 (at 0 0.9) (layer F.Fab) hide
       (effects (font (size 0.127 0.127) (thickness 0.03175)))
     )
@@
       (effects (font (size 0.8128 0.8128) (thickness 0.1524)))
     )
-    (fp_text value 100n (at 0 0.9) (layer F.Fab) hide
+    (fp_text value 2u2 (at 0 0.9) (layer F.Fab) hide
       (effects (font (size 0.127 0.127) (thickness 0.03175)))
     )
@@
       (effects (font (size 0.8128 0.8128) (thickness 0.1524)))
     )
-    (fp_text value 100n (at 0 0.9 90) (layer F.Fab) hide
+    (fp_text value 2u2 (at 0 0.9 90) (layer F.Fab) hide
       (effects (font (size 0.127 0.127) (thickness 0.03175)))
     )
@@
       (effects (font (size 0.8128 0.8128) (thickness 0.1524)))
     )
-    (fp_text value 100n (at 0 0.9) (layer F.Fab) hide
+    (fp_text value 2u2 (at 0 0.9) (layer F.Fab) hide
       (effects (font (size 0.127 0.127) (thickness 0.03175)))
     )
@@
       (effects (font (size 0.8128 0.8128) (thickness 0.1524)))
     )
-    (fp_text value 100n (at 0 0.9 90) (layer F.Fab) hide
+    (fp_text value 2u2 (at 0 0.9 90) (layer F.Fab) hide
       (effects (font (size 0.127 0.127) (thickness 0.03175)))
     )
@@
       (effects (font (size 0.8128 0.8128) (thickness 0.2032)))
     )
-    (fp_text value 33u (at 0 1.016) (layer F.Fab)
+    (fp_text value DNP (at 0 1.016) (layer F.Fab)
       (effects (font (size 0.508 0.508) (thickness 0.127)))
     )
@@
     (pad 1 smd roundrect (at -1.5375 0) (size 1.325 2.35) (layers F.Cu F.Paste F.Mask) (roundrect_rratio 0.188679)
       (net 1 +5V))
-    (model ${KISYS3DMOD}/Capacitor_Tantalum_SMD.3dshapes/CP_EIA-3528-21_Kemet-B.wrl
-      (at (xyz 0 0 0))
-      (scale (xyz 1 1 1))
-      (rotate (xyz 0 0 0))
-    )
   )
   (module stdpads:SOIC-16_7.5mm (layer F.Cu)
@@
     (pad 16 smd roundrect (at 4.65 -4.445) (size 2.05 0.6) (layers F.Cu F.Paste F.Mask) (roundrect_rratio 0.25)
       (net 1 +5V))
-    (model ${KISYS3DMOD}/Package_SO.3dshapes/SOIC-16W_7.5x10.3mm_P1.27mm.wrl
+    (model ${KISYS3DMOD}/Package_SO.3dshapes/SOIC-16W_7.5x10.3mm_P1.27mm.step
       (at (xyz 0 0 0))
       (scale (xyz 1 1 1))
@@
       (effects (font (size 0.8128 0.8128) (thickness 0.1524)))
     )
-    (fp_text value 100n (at 0 0.9) (layer F.Fab) hide
+    (fp_text value 2u2 (at 0 0.9) (layer F.Fab) hide
       (effects (font (size 0.127 0.127) (thickness 0.03175)))
     )
@@
       (effects (font (size 0.8128 0.8128) (thickness 0.2032)))
     )
-    (fp_text value 33u (at 0 1.016 90) (layer F.Fab)
+    (fp_text value DNP (at 0 1.016 90) (layer F.Fab)
       (effects (font (size 0.508 0.508) (thickness 0.127)))
     )
@@
     (pad 1 smd roundrect (at -1.5375 0 270) (size 1.325 2.35) (layers F.Cu F.Paste F.Mask) (roundrect_rratio 0.188679)
       (net 1 +5V))
-    (model ${KISYS3DMOD}/Capacitor_Tantalum_SMD.3dshapes/CP_EIA-3528-21_Kemet-B.wrl
-      (at (xyz 0 0 0))
-      (scale (xyz 1 1 1))
-      (rotate (xyz 0 0 0))
-    )
   )
   (module stdpads:C_0805 (layer F.Cu)
@@
       (effects (font (size 0.8128 0.8128) (thickness 0.1524)))
     )
-    (fp_text value 100n (at 0 0.9) (layer F.Fab) hide
+    (fp_text value 2u2 (at 0 0.9) (layer F.Fab) hide
       (effects (font (size 0.127 0.127) (thickness 0.03175)))
     )
@@
       (effects (font (size 0.8128 0.8128) (thickness 0.1524)))
     )
-    (fp_text value 100n (at 0 0.9) (layer F.Fab) hide
+    (fp_text value 2u2 (at 0 0.9) (layer F.Fab) hide
       (effects (font (size 0.127 0.127) (thickness 0.03175)))
     )
@@
       (effects (font (size 0.8128 0.8128) (thickness 0.2032)))
     )
-    (fp_text value 33u (at 0 1.016) (layer F.Fab)
+    (fp_text value DNP (at 0 1.016) (layer F.Fab)
       (effects (font (size 0.508 0.508) (thickness 0.127)))
     )
@@
     (pad 2 smd roundrect (at 1.5375 0 180) (size 1.325 2.35) (layers F.Cu F.Paste F.Mask) (roundrect_rratio 0.188679)
       (net 2 GND))
-    (model ${KISYS3DMOD}/Capacitor_Tantalum_SMD.3dshapes/CP_EIA-3528-21_Kemet-B.wrl
-      (at (xyz 0 0 0))
-      (scale (xyz 1 1 1))
-      (rotate (xyz 0 0 0))
-    )
   )
   (module stdpads:TSOP-II-44_400mil_P0.8mm (layer F.Cu)
@@
     (pad 44 smd roundrect (at 5.5875 -8.4 90) (size 1.525 0.55) (layers F.Cu F.Paste F.Mask) (roundrect_rratio 0.25)
       (net 62 /RA5))
-    (model ${KISYS3DMOD}/Package_SO.3dshapes/TSOP-II-44_10.16x18.41mm_P0.8mm.wrl
-      (at (xyz 0 0 0))
-      (scale (xyz 1 1 1))
+    (model ${KISYS3DMOD}/Package_SO.3dshapes/TSOP-II-44_10.16x18.41mm_P0.8mm.step
+      (at (xyz 0 0 0))
+      (scale (xyz 1 1 1))

Commit message: Removed AVR-JTAG-10 connector footprint
Parts:
- U2: value DS1215 -> DS1315S-5
Changed lines of the file:
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@@
-(kicad_pcb (version 20171130) (host pcbnew "(5.1.2-1)-1")
+(kicad_pcb (version 20171130) (host pcbnew "(5.1.5-0-10_14)")
   (general
     (thickness 1.6)
@@
       (effects (font (size 0.8128 0.8128) (thickness 0.2032)))
     )
-    (fp_text value DS1215 (at 0 1.27) (layer F.Fab)
+    (fp_text value DS1315S-5 (at 0 1.27) (layer F.Fab)
       (effects (font (size 0.8128 0.8128) (thickness 0.2032)))
     )
